File: pcb/fortemis_left.kicad_pcb (KiCad board)
At the start: 2 copper layers, 124.2 x 100.8 mm, 26 parts

Commit message: Rebuild PCBs and fab files for the new thumbs
Parts:
- moved S17 27.4 mm to (109.5, 37.2), turned to -56.162 degrees
- moved S16 26.2 mm to (96.2, 22.1), turned to -41.162 degrees
- moved S15 24.4 mm to (79.5, 10.9), turned to -26.162 degrees
- moved NUT5 23.7 mm to (107.7, 48.6), turned to -56.162 degrees
Routing:
- net GND: track 0.00 -> 368.4 mm, vias 93 -> 109
- net D11: track 146.7 -> 187.7 mm, vias 2 -> 8
- net D0: track 176.1 -> 216.0 mm, vias 4 -> 10
- net BAT_P: track 46.8 -> 84.0 mm, vias 2 -> 3
- net D1: track 127.3 -> 155.3 mm
- net D9: track 41.8 -> 59.2 mm, vias 0 -> 4
- net BAT_RAW: track 49.0 -> 36.9 mm, vias 2 -> 0
- net D4: track 64.0 -> 74.7 mm, vias 2 -> 4
- net D17: track 31.1 -> 24.0 mm
- net D6: track 46.3 -> 52.7 mm, vias 2 -> 4
- net D5: track 63.2 -> 69.6 mm, vias 2 -> 4
- net D14: track 73.4 -> 79.5 mm
- net D2: track 107.6 -> 103.3 mm
- net D7: track 44.2 -> 47.7 mm, vias 0 -> 2
- net D12: track 116.9 -> 120.2 mm
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Other:
- board size 124.2 x 100.8 mm -> 145.3 x 119.6 mm
